File: moter_upgrade_boardv1.kicad_pcb (KiCad board)
At the start: 2 copper layers, 55 parts, among them J2 Conn_01x03_Socket, J3 Conn_01x02_Socket, J4 Conn_01x02_Socket, J5 Conn_01x02_Socket, J6 Conn_01x02_Socket, J7 Conn_ST_STDC14, J8 Conn_01x05_Socket, J9 USB_C_Receptacle_USB2.0_16P, SW1 SW_SPDT, SW2 SW_Push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

Commit message: test
Parts:
- removed C10, C6, C7, C8: 0.1uF, Capacitor_SMD:C_0603_1608Metric_Pad1.08x0.95mm_HandSolder
- removed C11: 0.1uf, Capacitor_SMD:C_0603_1608Metric_Pad1.08x0.95mm_HandSolder
- removed C12, C14: 1uf, Capacitor_SMD:C_0603_1608Metric_Pad1.08x0.95mm_HandSolder
- removed C4, C5: 2.2μF, Capacitor_SMD:C_0603_1608Metric_Pad1.08x0.95mm_HandSolder
- removed C9: 4.7uf, Capacitor_SMD:C_0805_2012Metric_Pad1.18x1.45mm_HandSolder
- removed D2: LED_GREEN, Capacitor_SMD:C_0603_1608Metric_Pad1.08x0.95mm_HandSolder
- removed J9: USB_C_Receptacle_USB2.0_16P, Connector_USB:USB_C_Receptacle_GCT_USB4105-xx-A_16P_TopMnt_Horizontal
- removed R10, R9: 5.1k, Resistor_SMD:R_0603_1608Metric_Pad0.98x0.95mm_HandSolder
- removed R7: 1k, Resistor_SMD:R_0603_1608Metric_Pad0.98x0.95mm_HandSolder
- removed SW2: SW_Push, Button_Switch_THT:SW_PUSH_6mm
- removed U4: STM32H523CCTx, Package_QFP:LQFP-48_7x7mm_P0.5mm
- removed U6: CH340E, Package_SO:MSOP-10_3x3mm_P0.5mm
- added C18: 0.1uf, Capacitor_SMD:C_0603_1608Metric_Pad1.08x0.95mm_HandSolder, F.Cu at (221.0, 91.7)
- added C19: 4.7μF, Capacitor_SMD:C_0603_1608Metric_Pad1.08x0.95mm_HandSolder, F.Cu at (221.0, 94.2)
- added C21: 0.1uF, Capacitor_SMD:C_0603_1608Metric, B.Cu at (199.1, 138.1)
- added C22: 0.1uF, Capacitor_SMD:C_0603_1608Metric, B.Cu at (199.1, 140.0)
- added C23: 0.1uF, Capacitor_SMD:C_0603_1608Metric, B.Cu at (199.1, 142.0)
- added C24: 4.7uf, Capacitor_SMD:C_0603_1608Metric_Pad1.08x0.95mm_HandSolder, F.Cu at (221.0, 96.7)
- added C25: 0.1uF, Capacitor_SMD:C_0603_1608Metric, B.Cu at (199.1, 144.0)
- added C26: 0.1uf, Capacitor_SMD:C_0603_1608Metric, B.Cu at (199.1, 145.9)
- added C27: 1uf, Capacitor_SMD:C_0603_1608Metric, F.Cu at (221.0, 99.2)
- added D6: LED_YELLOW, Diode_SMD:D_0805_2012Metric_Pad1.15x1.40mm_HandSolder, F.Cu at (229.8, 116.2)
- added R12: 1k, Resistor_SMD:R_0603_1608Metric_Pad0.98x0.95mm_HandSolder, F.Cu at (246.7, 121.3)
- added SW4: SW_Push, Button_Switch_THT:SW_PUSH_6mm, F.Cu at (218.9, 116.8)
- added U8: STM32C542CCT6, Package_QFP:LQFP-64_10x10mm_P0.5mm, F.Cu at (125.4, 107.3)
- C13, D1, R1, R2, R3, R4, R5, R6, R8: moved to F.Cu
- moved G*** 216.0 mm to (243.6, 29.5)
- moved J5 167.5 mm to (212.8, 92.8), turned to 0 degrees
- moved J4 156.4 mm to (203.4, 92.8), turned to 0 degrees
- moved R8 136.1 mm to (251.0, 100.5)
- moved J6 118.6 mm to (217.3, 60.5), turned to -90 degrees
- moved J7 118.4 mm to (229.7, 103.1)
- moved D4 118.3 mm to (225.3, 89.2)
- moved R5 106.7 mm to (229.7, 89.2)
- moved JP1 105.8 mm to (204.9, 50.4)
- moved U7 102.9 mm to (223.1, 83.4), turned to 0 degrees
- moved SW1 101.4 mm to (205.7, 117.0)
- moved R2 100.5 mm to (225.3, 94.2)
- moved R4 99.3 mm to (225.3, 99.2)
- moved C13 99.0 mm to (221.0, 89.2), turned to 0 degrees
- moved R1 94.7 mm to (225.3, 91.7)
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Connections:
- J5 pad 1: CAN_L -> CAN_H
- J5 pad 2: CAN_H -> CAN_L
- J7 pad 12: trst -> njtrst
Routing:
- net +3.3V: track 37.7 -> 0.00 mm, vias 5 -> 0
- net uart1-rx: track 12.7 -> 0.00 mm
- net swdio: track 10.9 -> 0.00 mm
- net uart1-tx: track 10.0 -> 0.00 mm, vias 1 -> 0
- net trst: track 6.73 -> 0.00 mm
- net jtdi: track 6.73 -> 0.00 mm, vias 1 -> 0
- net swclk: track 6.04 -> 0.00 mm
- net swo: track 6.01 -> 0.00 mm
- net BOOT0: track 4.28 -> 0.00 mm, vias 1 -> 0
- net Net-(C5-Pad2): track 1.38 -> 0.00 mm, vias 1 -> 0
- net Net-(C4-Pad2): track 1.33 -> 0.00 mm, vias 1 -> 0
- net Net-(U6-V3): track 0.48 -> 0.00 mm, vias 1 -> 0

Commit message: 一応
バックアップ的な感じ
Parts:
- removed C13: 0.1uf, Capacitor_SMD:C_0603_1608Metric_Pad1.08x0.95mm_HandSolder
- removed J4, J5: Conn_01x02_Socket, Connector_JST:JST_XH_S2B-XH-A-1_1x02_P2.50mm_Horizontal
- removed JP1: Jumper_3_Bridged12, Connector_PinSocket_2.54mm:PinSocket_1x03_P2.54mm_Vertical
- removed R6: 120, Resistor_SMD:R_0603_1608Metric_Pad0.98x0.95mm_HandSolder
- removed SW3: SW_Wuerth_450301014042, Button_Switch_THT:SW_Slide-03_Wuerth-WS-SLTV_10x2.5x6.4_P2.54mm
- removed U5: MCP2562-E-P, Package_DIP:DIP-8_W7.62mm
- added C28: 0.1uF, Capacitor_SMD:C_0603_1608Metric_Pad1.08x0.95mm_HandSolder, F.Cu at (124.6, 109.8)
- added C29: 4.7uF, Capacitor_SMD:C_0603_1608Metric_Pad1.08x0.95mm_HandSolder, F.Cu at (124.6, 112.3)
- added C4: 4.7μF, Capacitor_SMD:C_0805_2012Metric_Pad1.18x1.45mm_HandSolder, F.Cu at (120.0, 98.0)
- added C5: 4.7μF, Capacitor_SMD:C_0805_2012Metric_Pad1.18x1.45mm_HandSolder, F.Cu at (120.0, 101.0)
- added C6: 22μF, Capacitor_SMD:C_0805_2012Metric_Pad1.18x1.45mm_HandSolder, F.Cu at (120.0, 104.0)
- added D2: D_Shockley, Diode_SMD:D_SOD-323_HandSoldering, F.Cu at (100.1, 110.2)
- added J12: Conn_01x02_Socket, Connector_JST:JST_XH_S2B-XH-A-1_1x02_P2.50mm_Horizontal, F.Cu at (121.1, 78.9)
- added J13: Conn_01x02_Socket, Connector_JST:JST_XH_S2B-XH-A-1_1x02_P2.50mm_Horizontal, F.Cu at (130.6, 78.9)
- added R11: 120, Resistor_SMD:R_0603_1608Metric_Pad0.98x0.95mm_HandSolder, F.Cu at (133.3, 107.3)
- added SW6: SW_Wuerth_450301014042, Button_Switch_THT:SW_Slide-03_Wuerth-WS-SLTV_10x2.5x6.4_P2.54mm, F.Cu at (142.3, 80.0)
- added U4: TCAN3414DRBR, TCAN3414DRBR:XCVR_TCAN3414DRBR, F.Cu at (108.6, 109.3)
- added U6: BD50FC0FP, Package_TO_SOT_SMD:TO-252-2, F.Cu at (112.4, 86.3)
- C1, C15, C16, C17, C2, C21, C22, C23, C25, C26, C3: moved to F.Cu
- moved C27 173.0 mm to (49.4, 77.2)
- moved C19 170.4 mm to (50.9, 83.0)
- moved C21 166.7 mm to (49.4, 64.7), turned to 0 degrees
- moved C22 166.5 mm to (49.4, 67.2), turned to 0 degrees
- moved C23 166.2 mm to (49.4, 69.7), turned to 0 degrees
- moved C25 166.0 mm to (49.4, 72.2), turned to 0 degrees
- moved C26 165.8 mm to (49.4, 74.7), turned to 0 degrees
- moved R8 117.8 mm to (133.3, 104.8)
- moved D6 116.6 mm to (113.5, 108.6)
- moved D1 114.3 mm to (100.1, 107.2)
- moved D3 114.1 mm to (100.1, 113.1)
- moved R12 114.0 mm to (133.3, 109.8)
- moved SW4 112.5 mm to (107.5, 100.5)
- moved U7 111.2 mm to (112.4, 94.5)
- moved R5 97.3 mm to (133.3, 102.3)
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